Commit message: partial progress, pushing in order to work from laptop

File: examples/jumping/five_link_biped.urdf (robot description, URDF)
Before this commit: robot KneedCompassGait, 14 links, 12 joints
Links:
- removed link hip
- link torso_mass: mass 2.5 -> 5
Joints:
- removed joint hip_pin
- removed joint left_leg_weld
- added joint left_hip_pin: type revolute, parent torso, child left_upper_leg, axis 0 1 0
- added joint right_hip_pin: type revolute, parent torso, child right_upper_leg, axis 0 1 0
- joint left_knee_pin: type continuous -> revolute
- joint planar_roty: child hip -> torso

Commit message: traj opt is running but getting bad results, need to take a look at mass/inertia values as well as constraints

File: examples/jumping/five_link_biped.urdf (robot description, URDF)
Before this commit: robot five_link_biped, 13 links, 12 joints
Links:
- link torso_mass: mass 5 -> 2.5
Joints:
- joint left_hip_pin: limit (none) -> effort=100; origin (none) -> xyz=0 0 0
- joint right_hip_pin: limit (none) -> effort=100; origin (none) -> xyz=0 0 0
- joint torso_mass_weld: origin (none) -> xyz=0 0 0.25

Commit message: successful knee bend, now working on implementing seeding initial conditions from previous trajectories

File: examples/jumping/five_link_biped.urdf (robot description, URDF)
Before this commit: robot five_link_biped, 13 links, 12 joints
Links:
- added link left_foot
- added link right_foot
- link left_lower_leg: geometry collision sphere radius=0; visual cylinder length=0.4 radius=0.0075
- link left_lower_leg_mass: mass 2.5 -> 3.2
- link left_upper_leg: geometry visual cylinder length=0.4 radius=0.0075
- link left_upper_leg_mass: mass 2.5 -> 6.4
- link right_lower_leg: geometry collision sphere radius=0; visual cylinder length=0.4 radius=0.0075
- link right_lower_leg_mass: mass 2.5 -> 3.2
- link right_upper_leg: geometry visual cylinder length=0.4 radius=0.0075
- link right_upper_leg_mass: mass 2.5 -> 6.4
- link torso: geometry visual cylinder length=0.625 radius=0.0075
- link torso_mass: mass 2.5 -> 12.0
Joints:
- added joint left_foot: type fixed, parent left_lower_leg, child left_foot, origin xyz=0 0 -.2
- added joint right_foot: type fixed, parent right_lower_leg, child right_foot, origin xyz=0 0 -.2
- joint left_knee_pin: origin xyz=0 0 -0.5 -> xyz=0 0 -0.4
- joint right_knee_pin: origin xyz=0 0 -0.5 -> xyz=0 0 -0.4
- joint torso_mass_weld: origin xyz=0 0 0.25 -> xyz=0 0 0.3125

Commit message: getting weird valid solutions in dircon

File: examples/jumping/five_link_biped.urdf (robot description, URDF)
Before this commit: robot rabbit, 15 links, 14 joints
Joints:
- joint left_foot: origin xyz=0 0 -.2 -> xyz=0 0 -.4
- joint right_foot: origin xyz=0 0 -.2 -> xyz=0 0 -.4

Commit message: working on osc - visualizer/sim work

File: examples/jumping/five_link_biped.urdf (robot description, URDF)
Before this commit: robot rabbit, 15 links, 14 joints
Links:
- link left_foot: geometry visual sphere radius=0.01
- link right_foot: geometry visual sphere radius=0.01

Commit message: jumping isn't stable

File: examples/jumping/five_link_biped.urdf (robot description, URDF)
Before this commit: robot rabbit, 15 links, 14 joints
Joints:
- joint left_hip_pin: limit effort=100 -> effort=200
- joint left_knee_pin: limit effort=100 -> effort=200
- joint right_hip_pin: limit effort=100 -> effort=200
- joint right_knee_pin: limit effort=100 -> effort=200

Commit message: figure out why ddy_des is off at time 1.5

File: examples/jumping/five_link_biped.urdf (robot description, URDF)
Before this commit: robot rabbit, 15 links, 14 joints
Joints:
- joint left_hip_pin: limit effort=200 -> effort=300
- joint left_knee_pin: limit effort=200 -> effort=300
- joint right_hip_pin: limit effort=200 -> effort=300
- joint right_knee_pin: limit effort=200 -> effort=300

Commit message: ddy_des in the z direction is too large, causing QP to fail

File: examples/jumping/five_link_biped.urdf (robot description, URDF)
Before this commit: robot rabbit, 15 links, 14 joints
Joints:
- joint left_hip_pin: limit effort=300 -> effort=1000
- joint left_knee_pin: limit effort=300 -> effort=1000
- joint right_hip_pin: limit effort=300 -> effort=1000
- joint right_knee_pin: limit effort=300 -> effort=1000

Commit message: increasing sim publish rate helps but need to look deeper still

File: examples/jumping/five_link_biped.urdf (robot description, URDF)
Before this commit: robot rabbit, 15 links, 14 joints
Joints:
- joint left_hip_pin: limit effort=1000 -> effort=300
- joint left_knee_pin: limit effort=1000 -> effort=300
- joint right_hip_pin: limit effort=1000 -> effort=300
- joint right_knee_pin: limit effort=1000 -> effort=300
