Commit message: Works for each 1 dof spine

File: examples/Spirit/spirit_cor_spine_drake.urdf (robot description, URDF)
Before this commit: robot spirit, 18 links, 17 joints
Joints:
- removed joint spine
- added joint cor_spine: type revolute, parent body, child body_front, origin xyz=0.08375 0 0, axis 1 0 0

File: examples/Spirit/xacros/spirit_sag_spine_drake.urdf.xacro (robot description, xacro)
@@ -141,5 +141,5 @@
 		</collision>
 	</link>
-	<joint name="spine" type="revolute">
+	<joint name="sag_spine" type="revolute">
 		<parent link="body"/>
 		<child link="body_front"/>
@@ -151,8 +151,8 @@
 	<transmission name="transmission_spine">
 		<type>transmission_interface/SimpleTransmission</type>
-		<joint name="spine">
+		<joint name="sag_spine">
 			<!-- <hardwareInterface>hardware_interface/EffortJointInterface</hardwareInterface> -->
 		</joint>
-		<actuator name="motor_spine">
+		<actuator name="motor_sag_spine">
 			<!-- <hardwareInterface>EffortJointInterface</hardwareInterface> -->
 			<mechanicalReduction>1</mechanicalReduction>
