Commit message: Update: spirit urdf

File: examples/Spirit/xacros/spirit_with_spine_drake.urdf (robot description, URDF)
Before this commit: robot spirit, 18 links, 17 joints
Joints:
- joint joint_12: limit lower=-1.570796326795 upper=1.570796326795 effort=1000 velocity=1000.00 -> lower=-0.707 upper=0.707 effort=40 velocity=30

File: examples/Spirit/xacros/spirit_with_spine_drake.urdf.xacro (robot description, xacro)
@@ -67,4 +67,7 @@
 	<xacro:property name="jointSpeedLimit" value="30"/>
 	<xacro:property name="jointEffortLimit" value="40"/>
+	<xacro:property name="spineKinLimit" value="0.707"/>
+	<xacro:property name="spineSpeedLimit" value="30"/>
+	<xacro:property name="spineEffortLimit" value="40"/>
 	<xacro:property name="bodyColor" value="darkgray"/>
 	<xacro:property name="hipColor" value="copper"/>
@@ -145,5 +148,5 @@
 			<axis xyz="1 0 0"/>
 			<origin xyz="${bodyLength/4} 0 0"/>
-			<limit upper="${pi/2}" lower="${-pi/2}" effort="1000" velocity="1000.00"/>
+			<limit upper="${spineKinLimit}" lower="${-spineKinLimit}" effort="${spineEffortLimit}" velocity="${spineSpeedLimit}"/>
 			<dynamics damping="0.0" friction="0.0"/>
 	</joint>

Commit message: Update: fix front hip position and add base link in the middle

File: examples/Spirit/xacros/spirit_with_spine_drake.urdf (robot description, URDF)
Before this commit: robot spirit, 18 links, 17 joints
Links:
- added link body, mass 5.75; collision box size=0.1675 0.24 0.104; visual box size=0.1675 0.24 0.104
- link base_link: mass 5.75 -> None; geometry 
Joints:
- added joint fixed_rear: type fixed, parent base_link, child body, origin xyz=-0.08375 0 0
- joint joint_11: parent base_link -> body
- joint joint_9: parent base_link -> body

File: examples/Spirit/xacros/spirit_with_spine_drake.urdf.xacro (robot description, xacro)
@@ -97,4 +97,7 @@
 	-->
 	<!-- First body segment-->
+	<link name="base_link">
+	</link>
+	<!-- First body segment-->
 	<link name="body">
 		<visual>
@@ -119,8 +122,14 @@
 		</collision>
 	</link>
+	<!-- Fixed rear body displacement -->
+		<joint name="fixed_rear" type="fixed">
+			<parent link="base_link"/>
+			<child link="body"/>
+			<origin xyz="${-bodyLength/4} 0 0"/>
+	</joint>
 	<!-- Second body segment-->
 	<link name="second_body_segment">
 		<visual>
-			<origin rpy="0 0 0" xyz="${bodyLength/4} 0 0"/>
+			<origin rpy="0 0 0" xyz="0 0 0"/>
 			<geometry>
 				<box size="${bodyLength/2} ${bodyWidth} ${bodyHeight}"/>
@@ -144,5 +153,5 @@
 	<!-- body twist joint. Joint name: 12 -->
 		<joint name="joint_12" type="revolute">
-			<parent link="body"/>
+			<parent link="base_link"/>
 			<child link="second_body_segment"/>
 			<axis xyz="1 0 0"/>
