Commit message: Update: correct toes position constraints in trot

File: examples/Spirit_spine/spirit_with_spine_drake.urdf (robot description, URDF)
Before this commit: robot spirit, 19 links, 18 joints
Joints:
- joint joint_0: limit lower=-6.28318530718 upper=6.28318530718 effort=40 velocity=30 -> lower=-6.28318530718 upper=6.28318530718 effort=40 velocity=8
- joint joint_1: limit lower=0 upper=3.14159265359 effort=40 velocity=30 -> lower=0 upper=3.14159265359 effort=40 velocity=8
- joint joint_10: limit lower=-0.707 upper=0.707 effort=40 velocity=30 -> lower=-0.707 upper=0.707 effort=40 velocity=8
- joint joint_11: limit lower=-0.707 upper=0.707 effort=40 velocity=30 -> lower=-0.707 upper=0.707 effort=40 velocity=8
- joint joint_12: limit lower=-0.707 upper=0.707 effort=40 velocity=30 -> lower=-0.707 upper=0.707 effort=40 velocity=8
- joint joint_2: limit lower=-6.28318530718 upper=6.28318530718 effort=40 velocity=30 -> lower=-6.28318530718 upper=6.28318530718 effort=40 velocity=8
- joint joint_3: limit lower=0 upper=3.14159265359 effort=40 velocity=30 -> lower=0 upper=3.14159265359 effort=40 velocity=8
- joint joint_4: limit lower=-6.28318530718 upper=6.28318530718 effort=40 velocity=30 -> lower=-6.28318530718 upper=6.28318530718 effort=40 velocity=8
- joint joint_5: limit lower=0 upper=3.14159265359 effort=40 velocity=30 -> lower=0 upper=3.14159265359 effort=40 velocity=8
- joint joint_6: limit lower=-6.28318530718 upper=6.28318530718 effort=40 velocity=30 -> lower=-6.28318530718 upper=6.28318530718 effort=40 velocity=8
- joint joint_7: limit lower=0 upper=3.14159265359 effort=40 velocity=30 -> lower=0 upper=3.14159265359 effort=40 velocity=8
- joint joint_8: limit lower=-0.707 upper=0.707 effort=40 velocity=30 -> lower=-0.707 upper=0.707 effort=40 velocity=8
- joint joint_9: limit lower=-0.707 upper=0.707 effort=40 velocity=30 -> lower=-0.707 upper=0.707 effort=40 velocity=8
